Commit message: [container] Refactoring

File: bebop_gazebo/urdf/bebop.urdf.xacro (robot description, xacro)
@@ -10,5 +10,5 @@
   <xacro:property name="wind_direction_z" value="$(arg wind_direction_z)" />
   <!-- Instantiate bebop "mechanics" -->
-  	<xacro:include filename="$(find med_uav_description)/urdf/bebop_base.urdf.xacro" />
+  	<xacro:include filename="$(find bebop_gazebo)/urdf/bebop_base.urdf.xacro" />
   	<xacro:include filename="$(find rotors_description)/urdf/component_snippets.xacro" />
   	<!-- Realistic odometry sensor with noise -->
@@ -72,22 +72,4 @@
 		<origin xyz="0.0 0.0 0.0" rpy="0.0 0.0 0.0" />
 	</xacro:odometry_plugin_macro>
-	<!-- Instantiate a wind plugin -->
-	<gazebo>
-	    <!-- wind plugin -->
-	    <plugin name="wind_plugin" filename="librotors_gazebo_wind_plugin.so">
-	      <robotNamespace>$(arg namespace)/</robotNamespace>
-	      <xyzOffset>0 0 0</xyzOffset>
-	      <frameId>base_link</frameId>
-	      <linkName>base_link</linkName>
-	      <windDirection>1 1 -0.3</windDirection>
-	      <windForceMean>0</windForceMean>
-	      <windForceVariance>0.0</windForceVariance>
-	      <windGustDirection>$(arg wind_direction_x) $(arg wind_direction_y) $(arg wind_direction_z)</windGustDirection>
-	      <windGustStart>$(arg wind_start)</windGustStart>
-	      <windGustDuration>$(arg wind_duration)</windGustDuration>
-	      <windGustForceMean>$(arg wind_force)</windGustForceMean>
-	      <windGustForceVariance>0</windGustForceVariance>
-	    </plugin>
-	</gazebo>
     <link name="laser1D_link">
       <inertial>

File: bebop_gazebo/urdf/bebop_base.urdf.xacro (robot description, xacro)
@@ -36,5 +36,5 @@
   </xacro:property>
   <!-- Included URDF Files -->
-  <xacro:include filename="$(find med_uav_description)/urdf/multirotor_base.urdf.xacro" />
+  <xacro:include filename="$(find bebop_gazebo)/urdf/multirotor_base.urdf.xacro" />
   <!-- Instantiate multirotor_base_macro once -->
   <xacro:multirotor_base_macro

File: bebop_gazebo/urdf/multirotor_base.urdf.xacro (robot description, xacro)
@@ -19,5 +19,5 @@
         <origin xyz="0 0 0" rpy="0 0 0" />
         <geometry>
-          <mesh filename="package://med_uav_description/meshes/${mesh_file}"
+          <mesh filename="package://bebop_gazebo/meshes/${mesh_file}"
             scale="0.001 0.001 0.001" />
           <!-- <box size="${body_width} ${body_width} ${body_height}"/> --> <!-- [m] [m] [m] -->
@@ -78,5 +78,5 @@
         <geometry>
           <!-- <cylinder length="0.005" radius="${radius_rotor}"/> --> <!-- [m] -->
-          <mesh filename="package://med_uav_description/meshes/propeller_${direction}.dae"
+          <mesh filename="package://bebop_gazebo/meshes/propeller_${direction}.dae"
             scale="0.00055 0.00055 0.00055" />
           <!-- <box size="${2*radius_rotor} 0.01 0.005"/> -->

File: bebop_gazebo/urdf/wind_turbine.base.urdf.xacro (robot description, xacro)
@@ -18,5 +18,5 @@
         <origin xyz="0 0 0" rpy="0 0 0" />
         <geometry>
-          <mesh filename="package://med_uav_description/meshes/wind_turbine_base.dae"
+          <mesh filename="package://bebop_gazebo/meshes/wind_turbine_base.dae"
             scale="2 2 2" />
         </geometry>
@@ -25,5 +25,5 @@
         <origin xyz="0 0 0" rpy="0 0 0"/>
         <geometry>
-          <mesh filename="package://med_uav_description/meshes/wind_turbine_base.dae"
+          <mesh filename="package://bebop_gazebo/meshes/wind_turbine_base.dae"
             scale="2 2 2" />
         </geometry>
@@ -45,5 +45,5 @@
         <origin xyz="0.16228 -0.00566 0.1" rpy="0 0 0" />
         <geometry>
-          <mesh filename="package://med_uav_description/meshes/wind_turbine_rotor.dae"
+          <mesh filename="package://bebop_gazebo/meshes/wind_turbine_rotor.dae"
             scale="2 2 2" />
         </geometry>
@@ -52,5 +52,5 @@
         <origin xyz="0.16228 -0.00566 0.1" rpy="0 0 0"/>
         <geometry>
-          <mesh filename="package://med_uav_description/meshes/wind_turbine_rotor.dae"
+          <mesh filename="package://bebop_gazebo/meshes/wind_turbine_rotor.dae"
             scale="2 2 2" />
         </geometry>

File: bebop_gazebo/urdf/wind_turbine.gazebo.xacro (robot description, xacro)
@@ -15,5 +15,5 @@
   <xacro:property name="bag_file" value="wind_turbine.bag" />
   <!-- Instantiate mmuav "mechanics" -->
-  <xacro:include filename="$(find med_uav_description)/urdf/wind_turbine.base.urdf.xacro" />
+  <xacro:include filename="$(find bebop_gazebo)/urdf/wind_turbine.base.urdf.xacro" />
   <xacro:include filename="$(find rotors_description)/urdf/component_snippets.xacro" />
 </robot>
