Commit message: [container] Add both small and big windturbines

File: bebop_gazebo/urdf/wind_turbine_big.base.urdf.xacro (robot description, xacro)
@@ -19,5 +19,5 @@
         <geometry>
           <mesh filename="package://bebop_gazebo/meshes/wind_turbine_base.dae"
-            scale="10 10 10" />
+            scale="100 100 100" />
         </geometry>
       </visual>
@@ -26,5 +26,5 @@
         <geometry>
           <mesh filename="package://bebop_gazebo/meshes/wind_turbine_base.dae"
-            scale="10 10 10" />
+            scale="100 100 100" />
         </geometry>
       </collision>
@@ -44,15 +44,15 @@
       </inertial>
       <visual>
-        <origin xyz="0.5 0 0" rpy="0 0 0" />
+        <origin xyz="0.5 0 0" rpy="${PI/2} 0 0" />
         <geometry>
           <mesh filename="package://bebop_gazebo/meshes/wind_turbine_rotor.dae"
-            scale="10 10 10" />
+            scale="100 100 100" />
         </geometry>
       </visual>
       <collision name='collision'>
-        <origin xyz="0.5 0 0" rpy="0 0 0"/>
+        <origin xyz="0.5 0 0" rpy="${PI/2} 0 0"/>
         <geometry>
           <mesh filename="package://bebop_gazebo/meshes/wind_turbine_rotor.dae"
-            scale="10 10 10" />
+            scale="100 100 100" />
         </geometry>
       </collision>
@@ -62,5 +62,5 @@
     <!--_____________________________________________________________-->
     <joint name="joint_wind_turbine_base" type="fixed">
-        <origin xyz="0 0 10.825" rpy="${PI/2} 0 0"/>
+        <origin xyz="0 0 50" rpy="0 0 0"/>
         <parent link="world"/>
         <child link="link_wind_turbine_rotor"/>
@@ -69,5 +69,6 @@
     <!--JOINT2 FIXED force_sensor_mount_top-->
     <!--_____________________________________________________________-->
-    <joint name="joint_wind_turbine_rotor" type="continuous">
+    <!--
+    <joint name="joint_wind_turbine_rotor" type="fixed">
         <origin xyz="1 0.0005 0.07" rpy="0 ${PI/2} 0" />
         <parent link="link_wind_turbine_base"/>
