Commit message: Resize wind turbine

File: bebop_gazebo/urdf/wind_turbine.base.urdf.xacro (robot description, xacro)
@@ -19,5 +19,5 @@
         <geometry>
           <mesh filename="package://bebop_gazebo/meshes/wind_turbine_base.dae"
-            scale="2 2 2" />
+            scale="10 10 10" />
         </geometry>
       </visual>
@@ -26,5 +26,5 @@
         <geometry>
           <mesh filename="package://bebop_gazebo/meshes/wind_turbine_base.dae"
-            scale="2 2 2" />
+            scale="10 10 10" />
         </geometry>
       </collision>
@@ -43,15 +43,15 @@
       </inertial>
       <visual>
-        <origin xyz="0.16228 -0.00566 0.1" rpy="0 0 0" />
+        <origin xyz="0.5 0 0" rpy="0 0 0" />
         <geometry>
           <mesh filename="package://bebop_gazebo/meshes/wind_turbine_rotor.dae"
-            scale="2 2 2" />
+            scale="10 10 10" />
         </geometry>
       </visual>
       <collision name='collision'>
-        <origin xyz="0.16228 -0.00566 0.1" rpy="0 0 0"/>
+        <origin xyz="0.5 0 0" rpy="0 0 0"/>
         <geometry>
           <mesh filename="package://bebop_gazebo/meshes/wind_turbine_rotor.dae"
-            scale="2 2 2" />
+            scale="10 10 10" />
         </geometry>
       </collision>
@@ -61,5 +61,5 @@
     <!--_____________________________________________________________-->
     <joint name="joint_wind_turbine_base" type="fixed">
-        <origin xyz="0 0 2.166" rpy="${PI/2} 0 0"/>
+        <origin xyz="0 0 10.825" rpy="${PI/2} 0 0"/>
         <parent link="world"/>
         <child link="link_wind_turbine_base"/>
@@ -69,5 +69,5 @@
     <!--_____________________________________________________________-->
     <joint name="joint_wind_turbine_rotor" type="continuous">
-        <origin xyz="0.10024 0.0005 0.07" rpy="0 ${PI/2} 0" />
+        <origin xyz="1 0.0005 0.07" rpy="0 ${PI/2} 0" />
         <parent link="link_wind_turbine_base"/>
         <child link="link_wind_turbine_rotor"/>

Commit message: [container] World changes

File: bebop_gazebo/urdf/wind_turbine.base.urdf.xacro (robot description, xacro)
@@ -6,5 +6,5 @@
     <!--LINK1 wind_turbine base-->
     <!--_____________________________________________________________-->
-    <link name='link_wind_turbine_base'>
+    <!-- <link name='link_wind_turbine_base'>
       <inertial>
         <mass value="50" />
@@ -19,5 +19,5 @@
         <geometry>
           <mesh filename="package://bebop_gazebo/meshes/wind_turbine_base.dae"
-            scale="10 10 10" />
+            scale="100 100 100" />
         </geometry>
       </visual>
@@ -26,8 +26,9 @@
         <geometry>
           <mesh filename="package://bebop_gazebo/meshes/wind_turbine_base.dae"
-            scale="10 10 10" />
+            scale="100 100 100" />
         </geometry>
       </collision>
     </link>
+-->
     <!--_____________________________________________________________-->
     <!--LINK2 wind_turbine rotor-->
@@ -43,15 +44,15 @@
       </inertial>
       <visual>
-        <origin xyz="0.5 0 0" rpy="0 0 0" />
+        <origin xyz="0.5 0 0" rpy="${PI/2} 0 0" />
         <geometry>
           <mesh filename="package://bebop_gazebo/meshes/wind_turbine_rotor.dae"
-            scale="10 10 10" />
+            scale="100 100 100" />
         </geometry>
       </visual>
       <collision name='collision'>
-        <origin xyz="0.5 0 0" rpy="0 0 0"/>
+        <origin xyz="0.5 0 0" rpy="${PI/2} 0 0"/>
         <geometry>
           <mesh filename="package://bebop_gazebo/meshes/wind_turbine_rotor.dae"
-            scale="10 10 10" />
+            scale="100 100 100" />
         </geometry>
       </collision>
@@ -61,12 +62,13 @@
     <!--_____________________________________________________________-->
     <joint name="joint_wind_turbine_base" type="fixed">
-        <origin xyz="0 0 10.825" rpy="${PI/2} 0 0"/>
+        <origin xyz="0 0 50" rpy="0 0 0"/>
         <parent link="world"/>
-        <child link="link_wind_turbine_base"/>
+        <child link="link_wind_turbine_rotor"/>
     </joint>
     <!--_____________________________________________________________-->
     <!--JOINT2 FIXED force_sensor_mount_top-->
     <!--_____________________________________________________________-->
-    <joint name="joint_wind_turbine_rotor" type="continuous">
+    <!--
+    <joint name="joint_wind_turbine_rotor" type="fixed">
         <origin xyz="1 0.0005 0.07" rpy="0 ${PI/2} 0" />
         <parent link="link_wind_turbine_base"/>
@@ -84,3 +86,4 @@
       </actuator>
     </transmission>
+  -->
 </robot>

Commit message: [container] Fix small wind-turbine spawning

File: bebop_gazebo/urdf/wind_turbine.base.urdf.xacro (robot description, xacro)
@@ -6,5 +6,5 @@
     <!--LINK1 wind_turbine base-->
     <!--_____________________________________________________________-->
-    <!-- <link name='link_wind_turbine_base'>
+    <link name='link_wind_turbine_base'>
       <inertial>
         <mass value="50" />
@@ -30,5 +30,4 @@
       </collision>
     </link>
--->
     <!--_____________________________________________________________-->
     <!--LINK2 wind_turbine rotor-->
@@ -64,5 +63,5 @@
         <origin xyz="0 0 10.825" rpy="${PI/2} 0 0"/>
         <parent link="world"/>
-        <child link="link_wind_turbine_rotor"/>
+        <child link="link_wind_turbine_base"/>
     </joint>
     <!--_____________________________________________________________-->
